File: BotSwitch.kicad_pcb (KiCad board)
At the start: 2 copper layers, 73.2 x 15.9 mm, 16 parts, among them J1 Batt_In, J2 Pogo_3p, J3 to_bott, J4 LED_conn, J5 Pogo_3p, J6 Conn_01x03_Pin, J7 Batt_In, J8 Conn_01x02_Pin, J9 Pogo_3p, SW1 Screw Switch

Commit message: Final?
Parts:
- removed H1: MountingHole, MountingHole:MountingHole_3.2mm_M3
- removed the H2 at (25.2, 55.9)
- removed the H2 at (75.7, 60.5)
- removed the H2 at (58.4, 56.2)
- removed J4: LED_conn, footprints:LED_Solder_SMD
- added H2: MountingHole, MountingHole:MountingHole_4.3mm_M4, F.Cu at (111.0, 6.53)
- added H3: MountingHole, MountingHole:MountingHole_4.3mm_M4, F.Cu at (99.5, 34.5)
- added H4: MountingHole, MountingHole:MountingHole_3.2mm_M3, F.Cu at (133.5, 34.5)
- R1: moved to B.Cu
- moved J5 97.2 mm to (127.5, 31.4), turned to -90 degrees
- moved J9 96.7 mm to (123.5, 31.4), turned to -90 degrees
- moved J8 91.3 mm to (139.5, 33.5), turned to 0 degrees
- moved J6 80.7 mm to (115.5, 32.0), turned to 0 degrees
- moved J7 69.5 mm to (109.5, 32.0), turned to -90 degrees
- moved R1 67.6 mm to (127.4, 2.93), turned to 180 degrees
- moved D1 66.8 mm to (122.5, 2.53)
- moved SW1 66.1 mm to (121.5, 7.03)
- moved J3 64.5 mm to (128.4, 9.54), turned to 90 degrees
- moved J1 64.3 mm to (115.0, 9.03)
- moved J2 64.1 mm to (118.0, 3.36)
Connections:
- D1 pad 1: Net-(D1-K) -> GND
- D1 pad 2: /Switched_PWR -> Net-(D1-A)
- R1 pad 1: GND -> /Switched_PWR
- R1 pad 2: Net-(D1-K) -> Net-(D1-A)
Routing:
- net Net-(J5-Pin_3): track 21.5 -> 31.6 mm
- net Net-(D1-K): track 8.80 -> 0.00 mm, vias 1 -> 0
- net /Switched_PWR: track 20.0 -> 14.9 mm, vias 1 -> 0
- net GND: track 43.8 -> 48.0 mm, vias 1 -> 0
- net Net-(J5-Pin_2): track 14.8 -> 18.3 mm
- net Net-(D1-A): track 0.00 -> 3.04 mm, vias 0 -> 1
- net /Cell2: track 11.5 -> 8.77 mm
- net /Cell1: track 3.86 -> 3.24 mm
- added copper zone on B.Cu, net (none)
- added copper zone on F.Cu, net (none)
Other:
- board size 73.2 x 15.9 mm -> 48 x 39 mm
- board text added: "C2"
- board text added: "G"
- board text added: "SW+"
- board text added: "lh"
