File: BotSwitch.kicad_pcb (KiCad board)
At the start: 2 copper layers, 48 x 39 mm, 14 parts, among them J1 Batt_In, J2 Pogo_3p, J3 to_bott, J5 Pogo_3p, J6 Conn_01x03_Pin, J7 Batt_In, J8 Conn_01x02_Pin, J9 Pogo_3p, SW1 Screw Switch

Commit message: Final final
Other:
- board text added: "LH"
- board text removed: "lh"
Changed lines of the file:
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@@
 	)
 	(setup
+		(stackup
+			(layer "F.SilkS"
+				(type "Top Silk Screen")
+			)
+			(layer "F.Paste"
+				(type "Top Solder Paste")
+			)
+			(layer "F.Mask"
+				(type "Top Solder Mask")
+				(thickness 0.01)
+			)
+			(layer "F.Cu"
+				(type "copper")
+				(thickness 0.035)
+			)
+			(layer "dielectric 1"
+				(type "core")
+				(thickness 1.51)
+				(material "FR4")
+				(epsilon_r 4.5)
+				(loss_tangent 0.02)
+			)
+			(layer "B.Cu"
+				(type "copper")
+				(thickness 0.035)
+			)
+			(layer "B.Mask"
+				(type "Bottom Solder Mask")
+				(thickness 0.01)
+			)
+			(layer "B.Paste"
+				(type "Bottom Solder Paste")
+			)
+			(layer "B.SilkS"
+				(type "Bottom Silk Screen")
+			)
+			(copper_finish "None")
+			(dielectric_constraints no)
+		)
 		(pad_to_mask_clearance 0)
 		(allow_soldermask_bridges_in_footprints no)
@@
 		(tags "resistor handsolder")
 		(property "Reference" "R1"
-			(at 0 1.65 360)
+			(at 0 1.65 0)
 			(layer "B.SilkS")
 			(hide yes)
@@
 		)
 		(property "Value" "R"
-			(at 0 -1.65 360)
+			(at 0 -1.65 0)
 			(layer "B.Fab")
 			(effects
@@
 		)
 		(fp_text user "${REFERENCE}"
-			(at 0 0 360)
+			(at 0 0 0)
 			(layer "B.Fab")
 			(effects
@@
 		)
 	)
+	(gr_line
+		(start 113.004 3.532)
+		(end 113.004 4.532)
+		(stroke
+			(width 0.1)
+			(type default)
+		)
+		(layer "F.SilkS")
+	)
+	(gr_line
+		(start 113.004 10.032)
+		(end 113.004 11.032)
+		(stroke
+			(width 0.1)
+			(type default)
+		)
+		(layer "F.SilkS")
+	)
+	(gr_line
+		(start 130.504 8.532)
+		(end 130.504 9.532)
+		(stroke
+			(width 0.1)
+			(type default)
+		)
+		(layer "F.SilkS")
+	)
+	(gr_line
+		(start 113.004 2.032)
+		(end 113.004 3.032)
+		(stroke
+			(width 0.1)
+			(type default)
+		)
+		(layer "F.SilkS")
+	)
+	(gr_line
+		(start 130.504 2.032)
+		(end 130.504 3.032)
+		(stroke
+			(width 0.1)
+			(type default)
+		)
+		(layer "F.SilkS")
+	)
+	(gr_line
+		(start 113.004 8.532)
+		(end 113.004 9.532)
+		(stroke
+			(width 0.1)
+			(type default)
+		)
+		(layer "F.SilkS")
+	)
+	(gr_line
+		(start 130.504 10.032)
+		(end 130.504 11.032)
+		(stroke
+			(width 0.1)
+			(type default)
+		)
+		(layer "F.SilkS")
+	)
+	(gr_line
+		(start 130.504 3.532)
+		(end 130.504 4.532)
+		(stroke
+			(width 0.1)
+			(type default)
+		)
+		(layer "F.SilkS")
+	)
 	(gr_arc
 		(start 142.503999 39.531999)
@@
 		)
 	)
-	(gr_text "lh"
-		(at 131.004 3.532 0)
+	(gr_text "LH"
+		(at 128.254 3.532 0)
 		(layer "F.SilkS")
 		(effects
@@
 			(xy 108.004 1.532) (xy 133.004 1.532)
 		)
-		(height -4.5)
+		(height -10.5)
 		(gr_text "25.0000 mm"
-			(at 120.504 -4.118 0)
+			(at 120.504 -10.118 0)
 			(layer "User.4")
 			(effects
@@
 		(layer "User.4")
 		(pts
-			(xy 105.504 11.532) (xy 105.504 1.532)
+			(xy 113.504 1.532) (xy 130.504 1.532)
+		)
+		(height -4.5)
+		(gr_text "17.0000 mm"
+			(at 122.004 -4.118 0)
+			(layer "User.4")
+			(effects
+				(font
+					(size 1 1)
+					(thickness 0.15)
+				)
+			)
+		)
+		(format
+			(prefix "")
+			(suffix "")
+			(units 3)
+			(units_format 1)
+			(precision 4)
+		)
+		(style
+			(thickness 0.1)
+			(arrow_length 1.27)
+			(text_position_mode 0)
+			(extension_height 0.58642)
+			(extension_offset 0.5) keep_text_aligned)
+	)
+	(dimension
+		(type aligned)
+		(layer "User.4")
+		(pts
+			(xy 108.004 11.532) (xy 108.004 1.532)
 		)
 		(height -4.5)
 		(gr_text "10.0000 mm"
-			(at 99.854 6.532 90)
+			(at 102.354 6.532 90)
 			(layer "User.4")
 			(effects
