File: BotSwitch.kicad_sch (KiCad schematic)
At the start: 17 parts, among them J1 Batt_In, J2 Pogo_3p, J3 to_bott, J4 LED_conn, J5 Pogo_3p, J6 Conn_01x03_Pin, J7 Batt_In, J8 Conn_01x02_Pin, J9 Pogo_3p, SW1 Screw Switch

Commit message: rm lock
Parts:
- removed H1: MountingHole, MountingHole:MountingHole_3.2mm_M3, symbol Mechanical:MountingHole
- removed J4: LED_conn, footprints:LED_Solder_SMD, symbol Connector:Conn_01x02_Pin
- removed R2: R, Resistor_SMD:R_0805_2012Metric_Pad1.20x1.40mm_HandSolder, symbol Device:R
